Commit message: "dynamics success"

File: src/robot_description/robot/urdf/robot.urdf (robot description, URDF)
Before this commit: robot robot, 18 links, 17 joints
Joints:
- joint leg1_joint2: origin xyz=0.0 -0.0993 0.0 rpy=0 0.785 0 -> xyz=0.0 -0.0993 0.0 rpy=0 0 0
- joint leg1_joint3: origin xyz=0.0 -0.0 -0.21 rpy=0 -2.355 0 -> xyz=0.0 -0.0 -0.21 rpy=0 0 0
- joint leg2_joint2: origin xyz=0.0 0.0993 0.0 rpy=0 0.785 0 -> xyz=0.0 0.0993 0.0 rpy=0 0 0
- joint leg2_joint3: origin xyz=0.0 0.0 -0.21 rpy=0 -2.355 0 -> xyz=0.0 0.0 -0.21 rpy=0 0 0
- joint leg3_joint2: origin xyz=-0.0 -0.0993 0.0 rpy=0 0.785 0 -> xyz=-0.0 -0.0993 0.0 rpy=0 0 0
- joint leg3_joint3: origin xyz=-0.0 -0.0 -0.21 rpy=0 -2.355 0 -> xyz=-0.0 -0.0 -0.21 rpy=0 0 0
- joint leg4_joint2: origin xyz=-0.0 0.0993 0.0 rpy=0 0.785 0 -> xyz=-0.0 0.0993 0.0 rpy=0 0 0
- joint leg4_joint3: origin xyz=-0.0 0.0 -0.21 rpy=0 -2.355 0 -> xyz=-0.0 0.0 -0.21 rpy=0 0 0
