Commit message: mpc success run wbc run but no adjust

File: src/robot_description/robot/urdf/leg.xacro (robot description, xacro)
@@ -172,7 +172,4 @@
         <parent link="${name}_link3" />
         <child link="${name}_link4" />
-        <axis xyz="0 0 0" />
-        <!-- <dynamics damping="0 friction="0"/>
-        <limit effort="0" velocity="0" lower="0" upper="0" /> -->
     </joint>
     <!--link4-->
@@ -211,4 +208,12 @@
                 <sphere radius="${collision_link4_radius}"/>
             </geometry>
+            <surface>
+                 <friction>
+                  <ode>
+                        <mu>1.0</mu>
+                        <mu2>1.0</mu2>
+                  </ode>
+                 </friction>
+            </surface>
         </collision>
     </link>

File: src/robot_description/robot/urdf/robot.xacro (robot description, xacro)
@@ -33,3 +33,117 @@
             </plugin>
         </gazebo>
+        <gazebo reference="base_link">
+            <mu1>0.2</mu1>
+            <mu2>0.2</mu2>
+            <kp  value="1000000.0"/>
+            <kd  value="1.0"/>
+        </gazebo>
+        <!--  leg 1-->
+        <gazebo reference="leg1_link1">
+            <mu1>0.2</mu1>
+            <mu2>0.2</mu2>
+            <material>Gazebo/DarkGrey</material>
+        </gazebo>
+        <gazebo reference="leg1_link2">
+            <mu1>0.2</mu1>
+            <mu2>0.2</mu2>
+            <self_collide>1</self_collide>
+            <material>Gazebo/DarkGrey</material>
+            <kp  value="1000000.0"/>
+            <kd  value="1.0"/>
+        </gazebo>
+        <gazebo reference="leg1_link3">
+            <mu1>0.2</mu1>
+            <mu2>0.2</mu2>
+            <self_collide>1</self_collide>
+        </gazebo>
+        <gazebo reference="leg1_link4">
+            <mu1>0.6</mu1>
+            <mu2>0.6</mu2>
+            <self_collide>1</self_collide>
+            <material>Gazebo/DarkGrey</material>
+            <kp  value="1000000.0"/>
+            <kd  value="1.0"/>
+        </gazebo>
+        <!--  leg 2-->
+        <gazebo reference="leg2_link1">
+            <mu1>0.2</mu1>
+            <mu2>0.2</mu2>
+            <material>Gazebo/DarkGrey</material>
+        </gazebo>
+        <gazebo reference="leg2_link2">
+            <mu1>0.2</mu1>
+            <mu2>0.2</mu2>
+            <self_collide>1</self_collide>
+            <material>Gazebo/DarkGrey</material>
+            <kp  value="1000000.0"/>
+            <kd  value="1.0"/>
+        </gazebo>
+        <gazebo reference="leg2_link3">
+            <mu1>0.2</mu1>
+            <mu2>0.2</mu2>
+            <self_collide>1</self_collide>
+        </gazebo>
+        <gazebo reference="leg2_link4">
+            <mu1>0.6</mu1>
+            <mu2>0.6</mu2>
+            <self_collide>1</self_collide>
+            <material>Gazebo/DarkGrey</material>
+            <kp  value="1000000.0"/>
+            <kd  value="1.0"/>
+        </gazebo>
+        <!--  leg 3-->
+        <gazebo reference="leg3_link1">
+            <mu1>0.2</mu1>
+            <mu2>0.2</mu2>
+            <material>Gazebo/DarkGrey</material>
+        </gazebo>
+        <gazebo reference="leg3_link2">
+            <mu1>0.2</mu1>
+            <mu2>0.2</mu2>
+            <self_collide>1</self_collide>
+            <material>Gazebo/DarkGrey</material>
+            <kp  value="1000000.0"/>
+            <kd  value="1.0"/>
+        </gazebo>
+        <gazebo reference="leg3_link3">
+            <mu1>0.2</mu1>
+            <mu2>0.2</mu2>
+            <self_collide>1</self_collide>
+        </gazebo>
+        <gazebo reference="leg3_link4">
+            <mu1>0.6</mu1>
+            <mu2>0.6</mu2>
+            <self_collide>1</self_collide>
+            <material>Gazebo/DarkGrey</material>
+            <kp  value="1000000.0"/>
+            <kd  value="1.0"/>
+        </gazebo>
+        <!--  leg 4-->
+        <gazebo reference="leg4_link1">
+            <mu1>0.2</mu1>
+            <mu2>0.2</mu2>
+            <material>Gazebo/DarkGrey</material>
+        </gazebo>
+        <gazebo reference="leg4_link2">
+            <mu1>0.2</mu1>
+            <mu2>0.2</mu2>
+            <self_collide>1</self_collide>
+            <material>Gazebo/DarkGrey</material>
+            <kp  value="1000000.0"/>
+            <kd  value="1.0"/>
+        </gazebo>
+        <gazebo reference="leg4_link3">
+            <mu1>0.2</mu1>
+            <mu2>0.2</mu2>
+            <self_collide>1</self_collide>
+        </gazebo>
+        <gazebo reference="leg4_link4">
+            <mu1>0.6</mu1>
+            <mu2>0.6</mu2>
+            <self_collide>1</self_collide>
+            <material>Gazebo/DarkGrey</material>
+            <kp  value="1000000.0"/>
+            <kd  value="1.0"/>
+        </gazebo>
 </robot>

File: src/robot_description/robot/urdf/robot_param.xacro (robot description, xacro)
@@ -10,6 +10,6 @@
     <!--电机的参数-->
         <!--前两个关节-->
-        <xacro:property name="motor1_damping" value="0.01"/>
-        <xacro:property name="motor1_friction" value="0.2"/>
+        <xacro:property name="motor1_damping" value="1e-1"/>
+        <xacro:property name="motor1_friction" value="1e-2"/>
         <xacro:property name="motor1_torque" value="36.0"/>
         <xacro:property name="motor1_vel" value="17.3"/>

Commit message: finial

File: src/robot_description/robot/urdf/leg.xacro (robot description, xacro)
@@ -105,5 +105,5 @@
         <collision>
             <origin
-                xyz="0 0 ${collision_link2_offest_z}" rpy="0 1.57 0" />
+                xyz="${collision_link2_offest_x} 0 ${collision_link2_offest_z}" rpy="0 1.657 0" />
             <geometry>
                 <box size="${collision_link2_length2} ${collision_link2_width} ${collision_link2_height}"/>
@@ -156,7 +156,7 @@
             <origin
                 xyz="0 0 ${collision_link3_offest_z}"
-                rpy="0 0 0" />
-            <geometry>
-                <cylinder length="${collision_link3_length}" radius="${collision_link3_radius}"/>
+                rpy="0 1.57 0" />
+            <geometry>
+                <box size="${collision_link3_length} ${collision_link3_width} ${collision_link3_height}"/>
             </geometry>
         </collision>

File: src/robot_description/robot/urdf/robot_param.xacro (robot description, xacro)
@@ -20,10 +20,10 @@
         <xacro:property name="motor2_vel" value="17.3"/>
         <!--关节角度限制 最小 最大-->
-        <xacro:property name="joint1_lb" value="-3.14"/>
-        <xacro:property name="joint1_ub" value="3.14"/>
-        <xacro:property name="joint2_lb" value="-3.14"/>
-        <xacro:property name="joint2_ub" value="3.14"/>
-        <xacro:property name="joint3_lb" value="-3.14"/>
-        <xacro:property name="joint3_ub" value="3.14"/>
+        <xacro:property name="joint1_lb" value="-0.75"/>
+        <xacro:property name="joint1_ub" value="0.75"/>
+        <xacro:property name="joint2_lb" value="-1.3"/>
+        <xacro:property name="joint2_ub" value="2.8"/>
+        <xacro:property name="joint3_lb" value="-2.805"/>
+        <xacro:property name="joint3_ub" value="-0.755"/>
     <!--body link-->
         <!--质量-->
@@ -65,5 +65,5 @@
         <!--joint2-->
             <!--关节初始偏移量 gazebo需要 mujoco不需要-->
-            <xacro:property name="joint2_offest_init" value="0.785"/> <!--45°-->
+            <xacro:property name="joint2_offest_init" value="0.0"/> <!--45°-->
             <!--关节相对父连杆的位置偏移-->
             <xacro:property name="joint2_offest_x" value="0.0"/>
@@ -86,5 +86,5 @@
         <!--joint3-->
             <!--关节初始偏移量 gazebo需要 mujoco不需要-->
-            <xacro:property name="joint3_offest_init" value="-2.355"/> <!---135°-->
+            <xacro:property name="joint3_offest_init" value="0.0"/> <!---135°-->
             <!--关节相对父连杆的位置偏移-->
             <xacro:property name="joint3_offest_x" value="0.0"/>
@@ -130,19 +130,21 @@
         <xacro:property name="collision_body_height" value="0.118"/>
     <!--link1 默认一个圆柱 长度 半径-->
-        <xacro:property name="collision_link1_length" value="0.06"/>
+        <xacro:property name="collision_link1_length" value="0.07"/>
         <xacro:property name="collision_link1_radius" value="0.038"/>
-        <xacro:property name="collision_link1_offest_y" value="-0.033"/>
+        <xacro:property name="collision_link1_offest_y" value="0.0"/>
     <!--link2 默认一个圆柱(长度 半径) 一个box（长宽高）-->
-        <xacro:property name="collision_link2_length1" value="0.117"/>
+        <xacro:property name="collision_link2_length1" value="0.07"/>
         <xacro:property name="collision_link2_radius" value="0.038"/>
-        <xacro:property name="collision_link2_offest_y" value="-0.036"/>
-        <xacro:property name="collision_link2_length2" value="0.165"/>
+        <xacro:property name="collision_link2_offest_y" value="-0.02"/>
+        <xacro:property name="collision_link2_length2" value="0.21"/>
         <xacro:property name="collision_link2_width" value="0.04"/>
-        <xacro:property name="collision_link2_height" value="0.06"/>
-        <xacro:property name="collision_link2_offest_z" value="-0.125"/>
+        <xacro:property name="collision_link2_height" value="0.04"/>
+        <xacro:property name="collision_link2_offest_z" value="-0.105"/>
+        <xacro:property name="collision_link2_offest_x" value="-0.02"/>
     <!--link3 默认一个圆柱 长度 半径-->
+        <xacro:property name="collision_link3_offest_z" value="-0.105"/>
         <xacro:property name="collision_link3_length" value="0.21"/>
-        <xacro:property name="collision_link3_radius" value="0.019"/>
-        <xacro:property name="collision_link3_offest_z" value="-0.105"/>
+        <xacro:property name="collision_link3_width" value="0.016"/>
+        <xacro:property name="collision_link3_height" value="0.016"/>
     <!--link4 默认一个球 半径-->
         <xacro:property name="collision_link4_radius" value="0.018"/>
